File: amp_board_Rev-A/amp_board_Rev-A.kicad_sch (KiCad schematic)
At the start: 6 parts, among them J10 V+_in, J12 GND, J7 V+_in

Commit message: Modified title block in schematic.
Other:
- title: (none) -> amp board
Changed lines of the file:
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@@
 	(generator_version "9.0")
 	(paper "A4")
+	(title_block
+		(title "amp board")
+		(date "2026-03-01")
+		(rev "A")
+	)
 	(wire
 		(pts
