File: amp_board_Rev-A/amp_section.kicad_sch (KiCad schematic)
At the start: 40 parts, among them J1 in, J11 in_GND, J2 R_power+, J3 R_power-, J4 MJ2955_E, J5 MJ2955_B, J6 MJ2955_C, J8 out, Q1 BC547, Q2 BC547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

Commit message: Modified title block in schematic.
Other:
- title: (none) -> amp board
Changed lines of the file:
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@@
 	(generator_version "9.0")
 	(paper "A4")
+	(title_block
+		(title "amp board")
+		(date "2026-03-01")
+		(rev "A")
+	)
 	(junction
 		(at 76.2 63.5)
